Commit message: passing real gripper config param by yaml file

File: wsg_50_simulation/urdf/wsg_50.urdf.xacro (robot description, xacro)
@@ -4,5 +4,5 @@
 <!-- finger_tip:    Offset of finger tip along fingers' motion direction.
                     Use e.g. for single contact point tip on finger. (default 0) -->
-<xacro:macro name="wsg_50_xacro" params="prefix parent finger_length finger_tip *origin sim_standalone:=false real_hardware:=false finger_type:='classic'">
+<xacro:macro name="wsg_50_xacro" params="prefix parent finger_length finger_tip *origin sim_standalone:=false real_hardware:=false finger_type:='classic' config_file:=${xacro.load_yaml('$(find wsg_50_driver)/config/wsg50_setup.yaml')}">
     <joint name="${prefix}_mounting_plate_joint" type="fixed">
         <xacro:insert_block name="origin"/>
@@ -308,13 +308,13 @@
             <hardware>
                 <plugin>wsg_50_interface::WSG50HardwareInterface</plugin>
-                <param name="gripper_name">wsg</param>
-                <param name="ip_address">192.168.1.20</param>
-                <param name="port">1000</param>
-                <param name="protocol">tcp</param>
-                <param name="local_port">1501</param>
-                <param name="rate">100.0</param>
-                <param name="grasping_force">10.0</param>
-                <param name="speed">20.</param>
-                <param name="finger_sensors">true</param>
+                <param name="gripper_name">${config_file.get('name')}</param>
+                <param name="ip_address">${config_file.get('ip_address')}</param>
+                <param name="port">${config_file.get('port')}</param>
+                <param name="protocol">${config_file.get('protocol')}</param>
+                <param name="local_port">${config_file.get('local_port')}</param>
+                <param name="rate">${config_file.get('rate')}</param>
+                <param name="grasping_force">${config_file.get('grasping_force')}</param>
+                <param name="speed">${config_file.get('speed')}</param>
+                <param name="finger_sensors">${config_file.get('finger_sensors')}</param>
             </hardware>
             <joint name="${prefix}_width_joint">

Commit message: Formalising the URDF for integration into our setup

File: wsg_50_simulation/urdf/wsg_50.urdf.xacro (robot description, xacro)
@@ -5,4 +5,10 @@
                     Use e.g. for single contact point tip on finger. (default 0) -->
 <xacro:macro name="wsg_50_xacro" params="prefix parent finger_length finger_tip *origin sim_standalone:=false real_hardware:=false finger_type:='classic' config_file:=${xacro.load_yaml('$(find wsg_50_driver)/config/wsg50_setup.yaml')}">
+    <link name="${prefix}_base"/>
+    <joint name="${prefix}_base_joint" type="fixed">
+        <origin xyz="0 0 0" rpy="0 0 0"/>
+        <parent link="${parent}"/>
+        <child link="${prefix}_base"/>
+    </joint>
     <joint name="${prefix}_mounting_plate_joint" type="fixed">
         <xacro:insert_block name="origin"/>
@@ -85,6 +91,6 @@
         <turnGravityOff>true</turnGravityOff>
     </gazebo>
-    <joint name="${prefix}_width_joint" type="prismatic">
-        <limit lower="0.002" upper="0.11" effort="100" velocity="100"/>
+    <joint name="${prefix}_joint" type="prismatic">
+        <limit lower="0.0" upper="0.11" effort="100" velocity="100"/>
         <origin xyz="0 0 0" rpy="0 -1.5708 0" />
         <parent link="${prefix}_base_link"/>
@@ -94,11 +100,11 @@
     <transmission name="${prefix}_base_trans" type="pr2_mechanism_model/SimpleTransmission">
         <actuator name="${prefix}_base_motor" />
-        <joint name="${prefix}_width_joint" />
+        <joint name="${prefix}_joint" />
         <mechanicalReduction>1</mechanicalReduction>
         <motorTorqueConstant>1</motorTorqueConstant>
     </transmission>
     <joint name="${prefix}_base_joint_gripper_left" type="prismatic">
-        <mimic joint="${prefix}_width_joint" multiplier="0.5" offset="0.0"/>
-        <limit lower="0.003" upper="0.055" effort="100" velocity="100"/>
+        <mimic joint="${prefix}_joint" multiplier="0.5" offset="0.0"/>
+        <limit lower="0.0" upper="0.055" effort="100" velocity="100"/>
         <origin xyz="0 0 0" rpy="0 0 0" />
         <parent link="${prefix}_base_link"/>
@@ -209,6 +215,6 @@
     <!-- GRIPPER RIGHT -->
     <joint name="${prefix}_base_joint_gripper_right" type="prismatic">
-        <mimic joint="${prefix}_width_joint" multiplier="0.5" offset="0.0"/>
-        <limit lower="0.003" upper="0.055" effort="100" velocity="100"/>
+        <mimic joint="${prefix}_joint" multiplier="0.5" offset="0.0"/>
+        <limit lower="0.0" upper="0.055" effort="100" velocity="100"/>
         <origin xyz="0 0 0" rpy="0 0 3.14159" />
         <parent link="${prefix}_base_link"/>
@@ -288,5 +294,5 @@
                 <plugin>gz_ros2_control/GazeboSimSystem</plugin>
             </hardware>
-            <joint name="${prefix}_width_joint">
+            <joint name="${prefix}_joint">
                 <command_interface name="velocity"/>
                 <command_interface name="position"/>
@@ -318,5 +324,5 @@
                 <param name="finger_sensors">${config_file.get('finger_sensors')}</param>
             </hardware>
-            <joint name="${prefix}_width_joint">
+            <joint name="${prefix}_joint">
                 <command_interface name="position"/>
                 <state_interface name="position"/>
