Commit message: rename package

File: wsg_50_simulation/urdf/wsg50.urdf.xacro (robot description, xacro)
@@ -2,7 +2,7 @@
 <robot name="wsg50" xmlns:xacro="http://www.ros.org/wiki/xacro">
     <!-- Import wsg50 macro -->
-    <xacro:include filename="$(find wsg50_simulation)/urdf/wsg_50.urdf.xacro" />
+    <xacro:include filename="$(find wsg_50_simulation)/urdf/wsg_50.urdf.xacro" />
     <link name="base_link"/>
-    <xacro:wsg_50_xacro name="wsg50" parent="base_link" finger_length="0.023" finger_tip="0.0">
+    <xacro:wsg_50_xacro prefix="wsg50" parent="base_link" finger_length="0.023" finger_tip="0.0">
         <origin xyz="0 0 0.1" rpy="0 0 0"/>
     </xacro:wsg_50_xacro>

File: wsg_50_simulation/urdf/wsg_50.urdf.xacro (robot description, xacro)
@@ -4,11 +4,11 @@
 <!-- finger_tip:    Offset of finger tip along fingers' motion direction.
                     Use e.g. for single contact point tip on finger. (default 0) -->
-<xacro:macro name="wsg_50_xacro" params="name parent finger_length finger_tip *origin">
-    <joint name="${name}_mounting_plate_joint" type="fixed">
+<xacro:macro name="wsg_50_xacro" params="prefix parent finger_length finger_tip *origin">
+    <joint name="${prefix}_mounting_plate_joint" type="fixed">
         <xacro:insert_block name="origin"/>
         <parent link="${parent}"/>
-        <child link="${name}_mounting_plate"/>
-    </joint>
-    <link name="${name}_mounting_plate">
+        <child link="${prefix}_mounting_plate"/>
+    </joint>
+    <link name="${prefix}_mounting_plate">
         <inertial>
             <mass value="0.25" />
@@ -19,5 +19,5 @@
             <origin xyz="0.0 0 0" rpy="0 0 0" />
             <geometry>
-                 <mesh filename="file://$(find wsg50_simulation)/meshes/FL_ISO50_WSG50.stl" scale="0.001 0.001 0.001"/>
+                 <mesh filename="file://$(find wsg_50_simulation)/meshes/FL_ISO50_WSG50.stl" scale="0.001 0.001 0.001"/>
             </geometry>
             <material name="black">
@@ -28,19 +28,19 @@
             <origin xyz="0.0 0 0" rpy="0 0 0" />
             <geometry>
-                 <mesh filename="file://$(find wsg50_simulation)/meshes/FL_ISO50_WSG50.stl" scale="0.001 0.001 0.001"/>
+                 <mesh filename="file://$(find wsg_50_simulation)/meshes/FL_ISO50_WSG50.stl" scale="0.001 0.001 0.001"/>
             </geometry>
          </collision>
     </link>
-    <!-- <gazebo reference="${name}_mounting_plate">
+    <!-- <gazebo reference="${prefix}_mounting_plate">
         <material>Gazebo/Grey</material>
         <turnGravityOff>true</turnGravityOff>
     </gazebo> -->
-    <joint name="${name}_anterior_gripper_joint" type="fixed">
-        <parent link="${name}_mounting_plate"/>
-        <child link="${name}_base_link"/>
+    <joint name="${prefix}_anterior_gripper_joint" type="fixed">
+        <parent link="${prefix}_mounting_plate"/>
+        <child link="${prefix}_base_link"/>
         <origin xyz="0 0 0" rpy="0 0 ${pi}" />
     </joint>
     <!-- BASE LINK -->
-    <link name="${name}_base_link">
+    <link name="${prefix}_base_link">
         <inertial>
             <mass value="0.25" />
@@ -54,5 +54,5 @@
             <origin xyz="0.0 0 0" rpy="0 0 0" />
             <geometry>
-                <mesh filename="file://$(find wsg50_simulation)/meshes/WSG50_110.stl" scale="1 1 1"/>
+                <mesh filename="file://$(find wsg_50_simulation)/meshes/WSG50_110.stl" scale="1 1 1"/>
             <!--box size="0.146 0.05 0.0735"/-->
             </geometry>
@@ -66,47 +66,47 @@
             <geometry>
             <!--box size="0.146 0.05 0.0735"/-->
-                <mesh filename="file://$(find wsg50_simulation)/meshes/WSG50_110.stl" scale="1 1 1"/>
-            </geometry>
-        </collision>
-    </link>
-    <gazebo reference="${name}_base_link">
+                <mesh filename="file://$(find wsg_50_simulation)/meshes/WSG50_110.stl" scale="1 1 1"/>
+            </geometry>
+        </collision>
+    </link>
+    <gazebo reference="${prefix}_base_link">
         <material>Gazebo/Grey</material>
         <turnGravityOff>true</turnGravityOff>
     </gazebo>
-    <joint name="${name}_center_joint" type="fixed">
+    <joint name="${prefix}_center_joint" type="fixed">
         <origin xyz="0 0 ${finger_length}" rpy="0 0 0" />      <!--origin xyz="-0.0067 0 0.049" rpy="0 0 0" /-->
-        <parent link="${name}_base_link"/>
-        <child link="${name}_center" />
-    </joint>
-    <link name="${name}_center">
+        <parent link="${prefix}_base_link"/>
+        <child link="${prefix}_center" />
+    </joint>
+    <link name="${prefix}_center">
     </link>
     <!-- GRIPPER LEFT -->
-    <joint name="${name}_base_joint_gripper_left" type="prismatic">
+    <joint name="${prefix}_base_joint_gripper_left" type="prismatic">
         <limit lower="-0.055" upper="-0.003" effort="1.0" velocity="1.0"/>
         <origin xyz="0 0 0" rpy="0 0 0" />      <!--origin xyz="-0.0067 0 0.049" rpy="0 0 0" /-->
-        <parent link="${name}_base_link"/>
-        <child link="${name}_gripper_left" />
+        <parent link="${prefix}_base_link"/>
+        <child link="${prefix}_gripper_left" />
         <!-- <dynamics friction="100" damping="100" /> -->
         <axis xyz="1 0 0"/>
         <limit effort="100" velocity="100"/>
     </joint>
-    <transmission name="${name}_base_trans_left" type="pr2_mechanism_model/SimpleTransmission">
-        <actuator name="${name}_base_motor_left" />
-        <joint name="${name}_base_joint_gripper_left" />
+    <transmission name="${prefix}_base_trans_left" type="pr2_mechanism_model/SimpleTransmission">
+        <actuator name="${prefix}_base_motor_left" />
+        <joint name="${prefix}_base_joint_gripper_left" />
         <mechanicalReduction>1</mechanicalReduction>
         <motorTorqueConstant>1</motorTorqueConstant>
     </transmission>
-    <link name="${name}_gripper_left">
-        <inertial>
-            <mass value="0.1" />
-            <origin xyz="0 0 0" />
-        <inertia ixx="1.0" ixy="0.0" ixz="0.0"
-                iyy="1.0" iyz="0.0"
-                izz="1.0" />
-        </inertial>
-        <visual>
-            <origin xyz="0.0 0 0" rpy="0 0 0" />
-            <geometry>
-                <mesh filename="file://$(find wsg50_simulation)/meshes/GUIDE_WSG50_110.stl" scale="0.001 0.001 0.001"/>
+    <link name="${prefix}_gripper_left">
+        <inertial>
+            <mass value="0.1" />
+            <origin xyz="0 0 0" />
+        <inertia ixx="1.0" ixy="0.0" ixz="0.0"
+                iyy="1.0" iyz="0.0"
+                izz="1.0" />
+        </inertial>
+        <visual>
+            <origin xyz="0.0 0 0" rpy="0 0 0" />
+            <geometry>
+                <mesh filename="file://$(find wsg_50_simulation)/meshes/GUIDE_WSG50_110.stl" scale="0.001 0.001 0.001"/>
             <!--box size="0.0175 0.03 0.024"/-->
             </geometry>
@@ -119,34 +119,34 @@
             <geometry>
             <!--box size="0.0175 0.03 0.024"/-->
-                <mesh filename="file://$(find wsg50_simulation)/meshes/GUIDE_WSG50_110.stl" scale="0.001 0.001 0.001"/>
-            </geometry>
-        </collision>
-        <contact_coefficients kd="1.0" kp="1000.0" mu="0"/>
-    </link>
-    <gazebo reference="${name}_gripper_left">
+                <mesh filename="file://$(find wsg_50_simulation)/meshes/GUIDE_WSG50_110.stl" scale="0.001 0.001 0.001"/>
+            </geometry>
+        </collision>
+        <contact_coefficients kd="1.0" kp="1000.0" mu="0"/>
+    </link>
+    <gazebo reference="${prefix}_gripper_left">
         <material>Gazebo/Blue</material>
         <turnGravityOff>true</turnGravityOff>
     </gazebo>
     <!-- LEFT FINGER -->
-    <joint name="${name}_guide_joint_finger_left" type="fixed">
+    <joint name="${prefix}_guide_joint_finger_left" type="fixed">
         <origin xyz="${finger_tip} 0 ${finger_length}" rpy="0 0 0" />
-        <parent link="${name}_gripper_left"/>
-        <child link="${name}_finger_left" />
+        <parent link="${prefix}_gripper_left"/>
+        <child link="${prefix}_finger_left" />
         <!-- <dynamics friction="100" damping="100" /> -->
         <axis xyz="1 0 0"/>
         <limit effort="100" velocity="100"/>
     </joint>
-    <link name="${name}_finger_left">
-        <inertial>
-            <mass value="0.1" />
-            <origin xyz="0 0 0" />
-        <inertia ixx="1.0" ixy="0.0" ixz="0.0"
-                iyy="1.0" iyz="0.0"
-                izz="1.0" />
-        </inertial>
-        <visual>
-            <origin xyz="0.0 0 0" rpy="0 0 0" />
-            <geometry>
-                <mesh filename="file://$(find wsg50_simulation)/meshes/WSG-FMF.stl" scale="0.001 0.001 0.001"/>
+    <link name="${prefix}_finger_left">
+        <inertial>
+            <mass value="0.1" />
+            <origin xyz="0 0 0" />
+        <inertia ixx="1.0" ixy="0.0" ixz="0.0"
+                iyy="1.0" iyz="0.0"
+                izz="1.0" />
+        </inertial>
+        <visual>
+            <origin xyz="0.0 0 0" rpy="0 0 0" />
+            <geometry>
+                <mesh filename="file://$(find wsg_50_simulation)/meshes/WSG-FMF.stl" scale="0.001 0.001 0.001"/>
             </geometry>
             <material name="black">
@@ -157,41 +157,41 @@
             <origin xyz="0 0 0" rpy="0 0 0" />
             <geometry>
-                <mesh filename="file://$(find wsg50_simulation)/meshes/WSG-FMF.stl" scale="0.001 0.001 0.001"/>
-            </geometry>
-        </collision>
-        <contact_coefficients kd="1.0" kp="1000.0" mu="0"/>
-    </link>
-    <gazebo reference="${name}_finger_left">
+                <mesh filename="file://$(find wsg_50_simulation)/meshes/WSG-FMF.stl" scale="0.001 0.001 0.001"/>
+            </geometry>
+        </collision>
+        <contact_coefficients kd="1.0" kp="1000.0" mu="0"/>
+    </link>
+    <gazebo reference="${prefix}_finger_left">
         <material>Gazebo/Blue</material>
         <turnGravityOff>true</turnGravityOff>
     </gazebo>
     <!-- GRIPPER RIGHT -->
-    <joint name="${name}_base_joint_gripper_right" type="prismatic">
+    <joint name="${prefix}_base_joint_gripper_right" type="prismatic">
         <limit lower="0.003" upper="0.055" effort="1.0" velocity="1.0"/>
         <origin xyz="0 0 0" rpy="0 0 3.14159" />
-        <parent link="${name}_base_link"/>
-        <child link="${name}_gripper_right" />
+        <parent link="${prefix}_base_link"/>
+        <child link="${prefix}_gripper_right" />
         <axis xyz="-1 0 0"/>
         <!-- <dynamics friction="100" damping="100" /> -->
         <limit effort="100" velocity="100"/>
     </joint>
-    <transmission name="${name}_base_trans_right" type="pr2_mechanism_model/SimpleTransmission">
-        <actuator name="${name}_base_motor_right" />
-        <joint name="${name}_base_joint_gripper_right" />
+    <transmission name="${prefix}_base_trans_right" type="pr2_mechanism_model/SimpleTransmission">
+        <actuator name="${prefix}_base_motor_right" />
+        <joint name="${prefix}_base_joint_gripper_right" />
         <mechanicalReduction>1</mechanicalReduction>
         <motorTorqueConstant>1</motorTorqueConstant>
     </transmission>
-        <link name="${name}_gripper_right">
-        <inertial>
-            <mass value="0.1" />
-            <origin xyz="0 0 0" />
-        <inertia ixx="1.0" ixy="0.0" ixz="0.0"
-                iyy="1.0" iyz="0.0"
-                izz="1.0" />
-        </inertial>
-        <visual>
-            <origin xyz="0.0 0 0" rpy="0 0 0" />
-            <geometry>
-                <mesh filename="file://$(find wsg50_simulation)/meshes/GUIDE_WSG50_110.stl" scale="0.001 0.001 0.001"/>
+        <link name="${prefix}_gripper_right">
+        <inertial>
+            <mass value="0.1" />
+            <origin xyz="0 0 0" />
+        <inertia ixx="1.0" ixy="0.0" ixz="0.0"
+                iyy="1.0" iyz="0.0"
+                izz="1.0" />
+        </inertial>
+        <visual>
+            <origin xyz="0.0 0 0" rpy="0 0 0" />
+            <geometry>
+                <mesh filename="file://$(find wsg_50_simulation)/meshes/GUIDE_WSG50_110.stl" scale="0.001 0.001 0.001"/>
             <!--box size="0.0175 0.03 0.024"/-->
             </geometry>
@@ -204,5 +204,5 @@
             <geometry>
             <!--box size="0.0175 0.03 0.024"/-->
-                <mesh filename="file://$(find wsg50_simulation)/meshes/GUIDE_WSG50_110.stl" scale="0.001 0.001 0.001"/>
+                <mesh filename="file://$(find wsg_50_simulation)/meshes/GUIDE_WSG50_110.stl" scale="0.001 0.001 0.001"/>
             </geometry>
         </collision>
@@ -214,24 +214,24 @@
     </gazebo>
     <!-- RIGHT FINGER -->
-    <joint name="${name}_guide_joint_finger_right" type="fixed">
+    <joint name="${prefix}_guide_joint_finger_right" type="fixed">
         <origin xyz="${finger_tip} 0 ${finger_length}" rpy="0 0 0" />
-        <parent link="${name}_gripper_right"/>
-        <child link="${name}_finger_right" />
+        <parent link="${prefix}_gripper_right"/>
+        <child link="${prefix}_finger_right" />
         <!-- <dynamics friction="100" damping="100" /> -->
         <axis xyz="1 0 0"/>
         <limit effort="100" velocity="100"/>
     </joint>
-    <link name="${name}_finger_right">
-        <inertial>
-            <mass value="0.1" />
-            <origin xyz="0 0 0" />
-        <inertia ixx="1.0" ixy="0.0" ixz="0.0"
-                iyy="1.0" iyz="0.0"
-                izz="1.0" />
-        </inertial>
-        <visual>
-            <origin xyz="0.0 0 0" rpy="0 0 0" />
-            <geometry>
-                <mesh filename="file://$(find wsg50_simulation)/meshes/WSG-FMF.stl" scale="0.001 0.001 0.001"/>
+    <link name="${prefix}_finger_right">
+        <inertial>
+            <mass value="0.1" />
+            <origin xyz="0 0 0" />
+        <inertia ixx="1.0" ixy="0.0" ixz="0.0"
+                iyy="1.0" iyz="0.0"
+                izz="1.0" />
+        </inertial>
+        <visual>
+            <origin xyz="0.0 0 0" rpy="0 0 0" />
+            <geometry>
+                <mesh filename="file://$(find wsg_50_simulation)/meshes/WSG-FMF.stl" scale="0.001 0.001 0.001"/>
             </geometry>
             <material name="black">
@@ -242,18 +242,18 @@
             <origin xyz="0 0 0" rpy="0 0 0" />
             <geometry>
-                <mesh filename="file://$(find wsg50_simulation)/meshes/WSG-FMF.stl" scale="0.001 0.001 0.001"/>
-            </geometry>
-        </collision>
-        <contact_coefficients kd="1.0" kp="1000.0" mu="0"/>
-    </link>
-    <gazebo reference="${name}_finger_right">
+                <mesh filename="file://$(find wsg_50_simulation)/meshes/WSG-FMF.stl" scale="0.001 0.001 0.001"/>
+            </geometry>
+        </collision>
+        <contact_coefficients kd="1.0" kp="1000.0" mu="0"/>
+    </link>
+    <gazebo reference="${prefix}_finger_right">
         <material>Gazebo/White</material>
         <turnGravityOff>true</turnGravityOff>
     </gazebo>
-    <ros2_control name="${name}" type="actuator">
+    <ros2_control name="${prefix}" type="actuator">
         <hardware>
             <plugin>gz_ros2_control/GazeboSimSystem</plugin>
         </hardware>
-        <joint name="${name}_base_joint_gripper_right">
+        <joint name="${prefix}_base_joint_gripper_right">
             <command_interface name="position"/>
             <command_interface name="velocity"/>
@@ -264,5 +264,5 @@
             </state_interface>
         </joint>
-        <joint name="${name}_base_joint_gripper_left">
+        <joint name="${prefix}_base_joint_gripper_left">
             <command_interface name="velocity"/>
             <command_interface name="position"/>
@@ -276,5 +276,5 @@
   <!-- <gazebo>
       <plugin filename="gz_ros2_control-system" name="gz_ros2_control::GazeboSimROS2ControlPlugin">
-      <parameters>$(find wsg50_simulation)/controllers/wsg50_driver.yaml</parameters>
+      <parameters>$(find wsg_50_simulation)/controllers/wsg50_driver.yaml</parameters>
       </plugin>
   </gazebo> -->

Commit message: architectural review

File: wsg_50_simulation/urdf/wsg50.urdf.xacro (robot description, xacro)
@@ -4,5 +4,5 @@
     <xacro:include filename="$(find wsg_50_simulation)/urdf/wsg_50.urdf.xacro" />
     <link name="base_link"/>
-    <xacro:wsg_50_xacro prefix="wsg50" parent="base_link" finger_length="0.023" finger_tip="0.0">
+    <xacro:wsg_50_xacro prefix="wsg50" parent="base_link" finger_length="0.023" finger_tip="0.0" sim_standalone="true">
         <origin xyz="0 0 0.1" rpy="0 0 0"/>
     </xacro:wsg_50_xacro>

File: wsg_50_simulation/urdf/wsg_50.urdf.xacro (robot description, xacro)
@@ -4,5 +4,5 @@
 <!-- finger_tip:    Offset of finger tip along fingers' motion direction.
                     Use e.g. for single contact point tip on finger. (default 0) -->
-<xacro:macro name="wsg_50_xacro" params="prefix parent finger_length finger_tip *origin">
+<xacro:macro name="wsg_50_xacro" params="prefix parent finger_length finger_tip *origin sim_standalone:=false">
     <joint name="${prefix}_mounting_plate_joint" type="fixed">
         <xacro:insert_block name="origin"/>
@@ -274,9 +274,11 @@
         </joint>
     </ros2_control>
-  <!-- <gazebo>
-      <plugin filename="gz_ros2_control-system" name="gz_ros2_control::GazeboSimROS2ControlPlugin">
-      <parameters>$(find wsg_50_simulation)/controllers/wsg50_standalone.yaml</parameters>
-      </plugin>
-  </gazebo> -->
+    <xacro:if value="${sim_standalone}">
+        <gazebo>
+            <plugin filename="gz_ros2_control-system" name="gz_ros2_control::GazeboSimROS2ControlPlugin">
+                <parameters>$(find wsg_50_simulation)/controllers/wsg_50_standalone.yaml</parameters>
+            </plugin>
+        </gazebo>
+    </xacro:if>
 </xacro:macro>
 </robot>
