Commit message: add real wsg50 integration

File: wsg_50_simulation/urdf/wsg50.urdf.xacro (robot description, xacro)
@@ -1,8 +1,10 @@
 <?xml version="1.0"?>
 <robot name="wsg50" xmlns:xacro="http://www.ros.org/wiki/xacro">
+    <xacro:arg name="real_hardware" default="false"/>
+    <xacro:arg name="sim_standalone" default="true"/>
     <!-- Import wsg50 macro -->
     <xacro:include filename="$(find wsg_50_simulation)/urdf/wsg_50.urdf.xacro" />
     <link name="base_link"/>
-    <xacro:wsg_50_xacro prefix="wsg50" parent="base_link" finger_length="0.023" finger_tip="0.0" sim_standalone="true">
+    <xacro:wsg_50_xacro prefix="wsg50" parent="base_link" finger_length="0.023" finger_tip="0.0" sim_standalone="$(arg sim_standalone)" real_hardware="$(arg real_hardware)">
         <origin xyz="0 0 0.1" rpy="0 0 0"/>
     </xacro:wsg_50_xacro>

File: wsg_50_simulation/urdf/wsg_50.urdf.xacro (robot description, xacro)
@@ -4,5 +4,5 @@
 <!-- finger_tip:    Offset of finger tip along fingers' motion direction.
                     Use e.g. for single contact point tip on finger. (default 0) -->
-<xacro:macro name="wsg_50_xacro" params="prefix parent finger_length finger_tip *origin sim_standalone:=false">
+<xacro:macro name="wsg_50_xacro" params="prefix parent finger_length finger_tip *origin sim_standalone:=false real_hardware:=false finger_type:='classic'">
     <joint name="${prefix}_mounting_plate_joint" type="fixed">
         <xacro:insert_block name="origin"/>
@@ -12,7 +12,9 @@
     <link name="${prefix}_mounting_plate">
         <inertial>
-            <mass value="0.25" />
-            <origin xyz="0 0 -0.1" />
-        	  <inertia  ixx="1.0" ixy="0.0"  ixz="0.0"  iyy="1.0"  iyz="0.0"  izz="1.0" />
+            <mass value="0.13" />
+            <origin xyz="0 0 0" />
+                <inertia ixx="2.82e-5" ixy="0.0" ixz="0.0"
+                iyy="1.70e-4" iyz="0.0"
+                izz="1.96e-4"/>
         </inertial>
         <visual>
@@ -32,8 +34,4 @@
          </collision>
     </link>
-    <!-- <gazebo reference="${prefix}_mounting_plate">
-        <material>Gazebo/Grey</material>
-        <turnGravityOff>true</turnGravityOff>
-    </gazebo> -->
     <joint name="${prefix}_anterior_gripper_joint" type="fixed">
         <parent link="${prefix}_mounting_plate"/>
@@ -44,10 +42,7 @@
     <link name="${prefix}_base_link">
         <inertial>
-            <mass value="0.25" />
-            <origin xyz="0 0 0" />
-            <!--inertia ixx="1.0" ixy="0.0" ixz="0.0"
-                iyy="100.0" iyz="0.0"
-                izz="1.0" /-->
-            <inertia  ixx="1.0" ixy="0.0"  ixz="0.0"  iyy="1.0"  iyz="0.0"  izz="1.0" />
+            <mass value="1.1" />
+            <origin xyz="0 0 0.03625" />
+            <inertia ixx="7.11e-4" ixy="0.0" ixz="0.0" iyy="1.91e-3" iyz="0.0" izz="1.66e-3"/>
         </inertial>
         <visual>
@@ -55,7 +50,5 @@
             <geometry>
                 <mesh filename="file://$(find wsg_50_simulation)/meshes/WSG50_110.stl" scale="1 1 1"/>
-            <!--box size="0.146 0.05 0.0735"/-->
-            </geometry>
-            <!-- <material name="grey">-->
+            </geometry>
                 <material name="Robotiq-LightGrey">
                 <color rgba="1 1 1 1"/>
@@ -65,5 +58,4 @@
             <origin xyz="0.0 0 0" rpy="0 0 0" />
             <geometry>
-            <!--box size="0.146 0.05 0.0735"/-->
                 <mesh filename="file://$(find wsg_50_simulation)/meshes/WSG50_110.stl" scale="1 1 1"/>
             </geometry>
@@ -72,36 +64,55 @@
     <gazebo reference="${prefix}_base_link">
         <material>Gazebo/Grey</material>
-        <turnGravityOff>true</turnGravityOff>
     </gazebo>
     <joint name="${prefix}_center_joint" type="fixed">
-        <origin xyz="0 0 ${finger_length}" rpy="0 0 0" />      <!--origin xyz="-0.0067 0 0.049" rpy="0 0 0" /-->
+        <origin xyz="0 0 ${finger_length}" rpy="0 0 0" />
         <parent link="${prefix}_base_link"/>
         <child link="${prefix}_center" />
     </joint>
-    <link name="${prefix}_center">
-    </link>
-    <!-- GRIPPER LEFT -->
-    <joint name="${prefix}_base_joint_gripper_left" type="prismatic">
-        <limit lower="-0.055" upper="-0.003" effort="1.0" velocity="1.0"/>
-        <origin xyz="0 0 0" rpy="0 0 0" />      <!--origin xyz="-0.0067 0 0.049" rpy="0 0 0" /-->
+    <!-- Width LINK -->
+    <link name="${prefix}_center"/>
+    <link name ="${prefix}_width">
+        <inertial>
+            <mass value="0.01e-10" />
+            <origin xyz="0 0 0" />
+            <inertia ixx="0.0" ixy="0.0" ixz="0.0"
+                    iyy="0.0" iyz="0.0"
+                    izz="0.0" />
+        </inertial>
+    </link>
+     <gazebo reference="${prefix}_width">
+        <material>Gazebo/Red</material>
+        <turnGravityOff>true</turnGravityOff>
+    </gazebo>
+    <joint name="${prefix}_width_joint" type="prismatic">
+        <limit lower="0.002" upper="0.11" effort="100" velocity="100"/>
+        <origin xyz="0 0 0" rpy="0 -1.5708 0" />
         <parent link="${prefix}_base_link"/>
-        <child link="${prefix}_gripper_left" />
-        <!-- <dynamics friction="100" damping="100" /> -->
+        <child link="${prefix}_width" />
         <axis xyz="1 0 0"/>
-        <limit effort="100" velocity="100"/>
-    </joint>
-    <transmission name="${prefix}_base_trans_left" type="pr2_mechanism_model/SimpleTransmission">
-        <actuator name="${prefix}_base_motor_left" />
-        <joint name="${prefix}_base_joint_gripper_left" />
+    </joint>
+    <transmission name="${prefix}_base_trans" type="pr2_mechanism_model/SimpleTransmission">
+        <actuator name="${prefix}_base_motor" />
+        <joint name="${prefix}_width_joint" />
         <mechanicalReduction>1</mechanicalReduction>
         <motorTorqueConstant>1</motorTorqueConstant>
     </transmission>
+    <joint name="${prefix}_base_joint_gripper_left" type="prismatic">
+        <mimic joint="${prefix}_width_joint" multiplier="0.5" offset="0.0"/>
+        <limit lower="0.003" upper="0.055" effort="100" velocity="100"/>
+        <origin xyz="0 0 0" rpy="0 0 0" />
+        <parent link="${prefix}_base_link"/>
+        <child link="${prefix}_gripper_left" />
+        <axis xyz="-1 0 0"/>
+        <limit effort="100" velocity="100"/>
+        <dynamics friction="0" damping="25" />
+    </joint>
     <link name="${prefix}_gripper_left">
         <inertial>
-            <mass value="0.1" />
-            <origin xyz="0 0 0" />
-        <inertia ixx="1.0" ixy="0.0" ixz="0.0"
-                iyy="1.0" iyz="0.0"
-                izz="1.0" />
+            <mass value="0.03" />
+            <origin xyz="0 0 0.03625" />
+            <inertia ixx="3.81e-6" ixy="0.0" ixz="0.0"
+            iyy="2.37e-6" iyz="0.0"
+            izz="3.06e-6"/>
         </inertial>
         <visual>
@@ -109,5 +120,4 @@
             <geometry>
                 <mesh filename="file://$(find wsg_50_simulation)/meshes/GUIDE_WSG50_110.stl" scale="0.001 0.001 0.001"/>
-            <!--box size="0.0175 0.03 0.024"/-->
             </geometry>
             <material name="black">
@@ -118,5 +128,4 @@
             <origin xyz="0 0 0" rpy="0 0 0" />
             <geometry>
-            <!--box size="0.0175 0.03 0.024"/-->
                 <mesh filename="file://$(find wsg_50_simulation)/meshes/GUIDE_WSG50_110.stl" scale="0.001 0.001 0.001"/>
             </geometry>
@@ -126,6 +135,39 @@
     <gazebo reference="${prefix}_gripper_left">
         <material>Gazebo/Blue</material>
-        <turnGravityOff>true</turnGravityOff>
-    </gazebo>
+    </gazebo>
+    <xacro:if value="${finger_type == 'soft'}">
+        <link name="${prefix}_soft_gripper_left">
+            <inertial>
+                <mass value="0.052" />
+                <origin xyz="0 0 0" />
+                <inertia ixx="2.50e-5" ixy="0.0" ixz="0.0"
+                iyy="2.50e-5" iyz="0.0"
+                izz="2.60e-6"/>
+            </inertial>
+            <visual>
+                <origin xyz="0 0 0" rpy="-1.5708 0 0" />
+                <geometry>
+                    <mesh filename="file://$(find wsg_50_simulation)/meshes/finger_holder.stl" scale="1. 1. 1."/>
+                </geometry>
+                <material name="Robotiq-LightGrey">
+                    <color rgba="1 1 1 1"/>
+                </material>
+            </visual>
+            <collision>
+                <origin xyz="0 0 0" rpy="-1.5708  0 0" />
+                <geometry>
+                    <mesh filename="file://$(find wsg_50_simulation)/meshes/finger_holder.stl" scale="1. 1. 1."/>
+                </geometry>
+            </collision>
+        </link>
+        <joint name="${prefix}_soft_gripper_left_joint" type="fixed">
+            <origin xyz="0 0 0" rpy="0 0 0" />
+            <parent link="${prefix}_gripper_left"/>
+            <child link="${prefix}_soft_gripper_left" />
+            <dynamics friction="100" damping="100" />
+            <axis xyz="1 0 0"/>
+            <limit effort="100" velocity="100"/>
+        </joint>
+    </xacro:if>
     <!-- LEFT FINGER -->
     <joint name="${prefix}_guide_joint_finger_left" type="fixed">
@@ -133,5 +175,5 @@
         <parent link="${prefix}_gripper_left"/>
         <child link="${prefix}_finger_left" />
-        <!-- <dynamics friction="100" damping="100" /> -->
+        <dynamics friction="100" damping="100" />
         <axis xyz="1 0 0"/>
         <limit effort="100" velocity="100"/>
@@ -139,9 +181,9 @@
     <link name="${prefix}_finger_left">
         <inertial>
-            <mass value="0.1" />
-            <origin xyz="0 0 0" />
-        <inertia ixx="1.0" ixy="0.0" ixz="0.0"
-                iyy="1.0" iyz="0.0"
-                izz="1.0" />
+            <mass value="0.052" />
+            <origin xyz="0 0 0.085" />
+            <inertia ixx="2.50e-5" ixy="0.0" ixz="0.0"
+            iyy="2.50e-5" iyz="0.0"
+            izz="2.60e-6"/>
         </inertial>
         <visual>
@@ -164,29 +206,23 @@
     <gazebo reference="${prefix}_finger_left">
         <material>Gazebo/Blue</material>
-        <turnGravityOff>true</turnGravityOff>
     </gazebo>
     <!-- GRIPPER RIGHT -->
     <joint name="${prefix}_base_joint_gripper_right" type="prismatic">
-        <limit lower="0.003" upper="0.055" effort="1.0" velocity="1.0"/>
+        <mimic joint="${prefix}_width_joint" multiplier="0.5" offset="0.0"/>
+        <limit lower="0.003" upper="0.055" effort="100" velocity="100"/>
         <origin xyz="0 0 0" rpy="0 0 3.14159" />
         <parent link="${prefix}_base_link"/>
         <child link="${prefix}_gripper_right" />
         <axis xyz="-1 0 0"/>
-        <!-- <dynamics friction="100" damping="100" /> -->
         <limit effort="100" velocity="100"/>
-    </joint>
-    <transmission name="${prefix}_base_trans_right" type="pr2_mechanism_model/SimpleTransmission">
-        <actuator name="${prefix}_base_motor_right" />
-        <joint name="${prefix}_base_joint_gripper_right" />
-        <mechanicalReduction>1</mechanicalReduction>
-        <motorTorqueConstant>1</motorTorqueConstant>
-    </transmission>
-        <link name="${prefix}_gripper_right">
-        <inertial>
-            <mass value="0.1" />
+        <dynamics friction="0" damping="25" />
+    </joint>
+    <link name="${prefix}_gripper_right">
+        <inertial>
+            <mass value="0.03" />
             <origin xyz="0 0 0" />
-        <inertia ixx="1.0" ixy="0.0" ixz="0.0"
-                iyy="1.0" iyz="0.0"
-                izz="1.0" />
+        <inertia ixx="3.81e-6" ixy="0.0" ixz="0.0"
+           iyy="2.37e-6" iyz="0.0"
+           izz="3.06e-6"/>
         </inertial>
         <visual>
@@ -194,5 +230,4 @@
             <geometry>
                 <mesh filename="file://$(find wsg_50_simulation)/meshes/GUIDE_WSG50_110.stl" scale="0.001 0.001 0.001"/>
-            <!--box size="0.0175 0.03 0.024"/-->
             </geometry>
             <material name="black">
@@ -203,5 +238,4 @@
             <origin xyz="0 0 0" rpy="0 0 0" />
             <geometry>
-            <!--box size="0.0175 0.03 0.024"/-->
                 <mesh filename="file://$(find wsg_50_simulation)/meshes/GUIDE_WSG50_110.stl" scale="0.001 0.001 0.001"/>
             </geometry>
@@ -211,5 +245,4 @@
     <gazebo reference="gripper_right">
         <material>Gazebo/White</material>
-        <turnGravityOff>true</turnGravityOff>
     </gazebo>
     <!-- RIGHT FINGER -->
@@ -218,5 +251,5 @@
         <parent link="${prefix}_gripper_right"/>
         <child link="${prefix}_finger_right" />
-        <!-- <dynamics friction="100" damping="100" /> -->
+        <dynamics friction="100" damping="100" />
         <axis xyz="1 0 0"/>
         <limit effort="100" velocity="100"/>
@@ -224,9 +257,9 @@
     <link name="${prefix}_finger_right">
         <inertial>
-            <mass value="0.1" />
-            <origin xyz="0 0 0" />
-        <inertia ixx="1.0" ixy="0.0" ixz="0.0"
-                iyy="1.0" iyz="0.0"
-                izz="1.0" />
+            <mass value="0.052" />
+            <origin xyz="0 0 0.075" />
+            <inertia ixx="2.50e-5" ixy="0.0" ixz="0.0"
+            iyy="2.50e-5" iyz="0.0"
+            izz="2.60e-6"/>
         </inertial>
         <visual>
@@ -249,28 +282,43 @@
     <gazebo reference="${prefix}_finger_right">
         <material>Gazebo/White</material>
-        <turnGravityOff>true</turnGravityOff>
-    </gazebo>
-    <ros2_control name="${prefix}" type="actuator">
-        <hardware>
-            <plugin>gz_ros2_control/GazeboSimSystem</plugin>
-        </hardware>
-        <joint name="${prefix}_base_joint_gripper_right">
-            <command_interface name="position"/>
-            <command_interface name="velocity"/>
-            <state_interface name="velocity"/>
-            <state_interface name="position">
-            <!-- initial position for the mock system and simulation to avoid fingers spanning into other parts-->
-                <param name="initial_value">0.025</param>
-            </state_interface>
-        </joint>
-        <joint name="${prefix}_base_joint_gripper_left">
-            <command_interface name="velocity"/>
-            <command_interface name="position"/>
-            <state_interface name="velocity"/>
-            <state_interface name="position">
-            <!-- initial position for the mock system and simulation to avoid fingers spanning into other parts -->
-                <param name="initial_value">-0.025</param>
-            </state_interface>
-        </joint>
+    </gazebo>
+    <ros2_control name="${prefix}" type="system">
+        <xacro:unless value="${real_hardware}">
+            <hardware>
+                <plugin>gz_ros2_control/GazeboSimSystem</plugin>
+            </hardware>
+            <joint name="${prefix}_width_joint">
+                <command_interface name="velocity"/>
+                <command_interface name="position"/>
+                <state_interface name="velocity"/>
+                <state_interface name="position">
+                    <param name="initial_value">0.05</param>
+                </state_interface>
+                <state_interface name="effort"/>
+            </joint>
+            <joint name="${prefix}_base_joint_gripper_left">
+                <state_interface name="position">
+                </state_interface>
+            </joint>
+            <joint name="${prefix}_base_joint_gripper_right">
+                <state_interface name="position"/>
+            </joint>
+        </xacro:unless>
+        <xacro:if value="${real_hardware}">
+            <hardware>
+                <plugin>wsg_50_control::WSG50HardwareInterface</plugin>
+                <param name="gripper_name">wsg</param>
+                <param name="ip_address">192.168.1.22</param>
+                <param name="port">1000</param>
+                <param name="rate">100.0</param>
+                <param name="grasping_force">10.0</param>
+            </hardware>
+            <joint name="${prefix}_width_joint">
+                <command_interface name="position"/>
+                <state_interface name="position"/>
+                <state_interface name="velocity"/>
+                <state_interface name="effort"/>
+            </joint>
+        </xacro:if>
     </ros2_control>
     <xacro:if value="${sim_standalone}">
