Commit message: add umi finger

File: wsg_50_simulation/urdf/wsg50.urdf.xacro (robot description, xacro)
@@ -6,5 +6,5 @@
     <xacro:include filename="$(find wsg_50_simulation)/urdf/wsg_50.urdf.xacro" />
     <link name="base_link"/>
-    <xacro:wsg_50_xacro prefix="wsg50" parent="base_link" finger_length="0.023" finger_tip="0.0" sim_standalone="$(arg sim_standalone)" real_hardware="$(arg real_hardware)">
+    <xacro:wsg_50_xacro prefix="wsg50" parent="base_link" finger_length="0.023" finger_tip="0.0" sim_standalone="$(arg sim_standalone)" real_hardware="$(arg real_hardware)" finger_type="soft">
         <origin xyz="0 0 0.1" rpy="0 0 0"/>
     </xacro:wsg_50_xacro>

File: wsg_50_simulation/urdf/wsg_50.urdf.xacro (robot description, xacro)
@@ -4,5 +4,5 @@
 <!-- finger_tip:    Offset of finger tip along fingers' motion direction.
                     Use e.g. for single contact point tip on finger. (default 0) -->
-<xacro:macro name="wsg_50_xacro" params="prefix parent finger_length finger_tip *origin sim_standalone:=false real_hardware:=false finger_type:='classic' config_file:=${xacro.load_yaml('$(find wsg_50_driver)/config/wsg50_setup.yaml')}">
+<xacro:macro name="wsg_50_xacro" params="prefix parent finger_length finger_tip *origin sim_standalone:=false real_hardware:=false finger_type:='soft' config_file:=${xacro.load_yaml('$(find wsg_50_driver)/config/wsg50_setup.yaml')}">
     <link name="${prefix}_base"/>
     <joint name="${prefix}_base_joint" type="fixed">
@@ -140,40 +140,6 @@
     </link>
     <gazebo reference="${prefix}_gripper_left">
-        <material>Gazebo/Blue</material>
+        <material>Gazebo/Black</material>
     </gazebo>
-    <xacro:if value="${finger_type == 'soft'}">
-        <link name="${prefix}_soft_gripper_left">
-            <inertial>
-                <mass value="0.052" />
-                <origin xyz="0 0 0" />
-                <inertia ixx="2.50e-5" ixy="0.0" ixz="0.0"
-                iyy="2.50e-5" iyz="0.0"
-                izz="2.60e-6"/>
-            </inertial>
-            <visual>
-                <origin xyz="0 0 0" rpy="-1.5708 0 0" />
-                <geometry>
-                    <mesh filename="file://$(find wsg_50_simulation)/meshes/finger_holder.stl" scale="1. 1. 1."/>
-                </geometry>
-                <material name="Robotiq-LightGrey">
-                    <color rgba="1 1 1 1"/>
-                </material>
-            </visual>
-            <collision>
-                <origin xyz="0 0 0" rpy="-1.5708  0 0" />
-                <geometry>
-                    <mesh filename="file://$(find wsg_50_simulation)/meshes/finger_holder.stl" scale="1. 1. 1."/>
-                </geometry>
-            </collision>
-        </link>
-        <joint name="${prefix}_soft_gripper_left_joint" type="fixed">
-            <origin xyz="0 0 0" rpy="0 0 0" />
-            <parent link="${prefix}_gripper_left"/>
-            <child link="${prefix}_soft_gripper_left" />
-            <dynamics friction="100" damping="100" />
-            <axis xyz="1 0 0"/>
-            <limit effort="100" velocity="100"/>
-        </joint>
-    </xacro:if>
     <!-- LEFT FINGER -->
     <joint name="${prefix}_guide_joint_finger_left" type="fixed">
@@ -185,32 +151,82 @@
         <limit effort="100" velocity="100"/>
     </joint>
-    <link name="${prefix}_finger_left">
-        <inertial>
-            <mass value="0.052" />
-            <origin xyz="0 0 0.085" />
-            <inertia ixx="2.50e-5" ixy="0.0" ixz="0.0"
-            iyy="2.50e-5" iyz="0.0"
-            izz="2.60e-6"/>
-        </inertial>
-        <visual>
-            <origin xyz="0.0 0 0" rpy="0 0 0" />
-            <geometry>
-                <mesh filename="file://$(find wsg_50_simulation)/meshes/WSG-FMF.stl" scale="0.001 0.001 0.001"/>
-            </geometry>
-            <material name="black">
-            <color rgba="0 0 0 1"/>
-            </material>
-        </visual>
-        <collision>
-            <origin xyz="0 0 0" rpy="0 0 0" />
-            <geometry>
-                <mesh filename="file://$(find wsg_50_simulation)/meshes/WSG-FMF.stl" scale="0.001 0.001 0.001"/>
-            </geometry>
-        </collision>
-        <contact_coefficients kd="1.0" kp="1000.0" mu="0"/>
-    </link>
-    <gazebo reference="${prefix}_finger_left">
-        <material>Gazebo/Blue</material>
-    </gazebo>
+    <xacro:unless value="${finger_type == 'soft'}">
+        <link name="${prefix}_finger_left">
+            <inertial>
+                <mass value="0.052" />
+                <origin xyz="0 0 0.085" />
+                <inertia ixx="2.50e-5" ixy="0.0" ixz="0.0"
+                iyy="2.50e-5" iyz="0.0"
+                izz="2.60e-6"/>
+            </inertial>
+            <visual>
+                <origin xyz="0.0 0 0" rpy="0 0 0" />
+                <geometry>
+                    <mesh filename="file://$(find wsg_50_simulation)/meshes/WSG-FMF.stl" scale="0.001 0.001 0.001"/>
+                </geometry>
+                <material name="black">
+                <color rgba="0 0 0 1"/>
+                </material>
+            </visual>
+            <collision>
+                <origin xyz="0 0 0" rpy="0 0 0" />
+                <geometry>
+                    <mesh filename="file://$(find wsg_50_simulation)/meshes/WSG-FMF.stl" scale="0.001 0.001 0.001"/>
+                </geometry>
+            </collision>
+            <contact_coefficients kd="1.0" kp="1000.0" mu="0"/>
+        </link>
+        <gazebo reference="${prefix}_finger_left">
+            <material>Gazebo/Black</material>
+        </gazebo>
+    </xacro:unless>
+    <xacro:if value="${finger_type == 'soft'}">
+        <link name="${prefix}_finger_left">
+            <inertial>
+                <mass value="0.052" />
+                <origin xyz="0 0 0" />
+                <inertia ixx="2.50e-5" ixy="0.0" ixz="0.0"
+                        iyy="2.50e-5" iyz="0.0"
+                        izz="2.60e-6"/>
+            </inertial>
+            <!-- Visual for finger_base -->
+            <visual>
+                <origin xyz="0 0 -0.023" rpy="-1.5708 0 0" />
+                <geometry>
+                    <mesh filename="file://$(find wsg_50_simulation)/meshes/finger_base.stl" scale="1. 1. 1."/>
+                </geometry>
+                <material name="orange">
+                    <color rgba="0.98 0.29 0.08 1"/>
+                </material>
+            </visual>
+            <!-- Visual for finger_body -->
+            <visual>
+                <origin xyz="0 0.013 0.078" rpy="3.14 0 3.14" />
+                <geometry>
+                    <mesh filename="file://$(find wsg_50_simulation)/meshes/finger_body.stl" scale="1. 1. 1."/>
+                </geometry>
+                <material name="orange">
+                    <color rgba="0.98 0.29 0.08 1"/>
+                </material>
+            </visual>
+            <!-- Collision -->
+            <collision>
+                <origin xyz="0 0 -0.023" rpy="-1.5708 0 0" />
+                <geometry>
+                    <mesh filename="file://$(find wsg_50_simulation)/meshes/finger_base.stl" scale="1. 1. 1."/>
+                </geometry>
+            </collision>
+            <collision>
+                <origin xyz="0 0.013 0.078" rpy="3.14 0 3.14" />
+                <geometry>
+                    <mesh filename="file://$(find wsg_50_simulation)/meshes/finger_body.stl" scale="1. 1. 1."/>
+                </geometry>
+            </collision>
+            <contact_coefficients kd="1.0" kp="1000.0" mu="0"/>
+        </link>
+        <gazebo reference="${prefix}_finger_left">
+            <material>Gazebo/Orange</material>
+        </gazebo>
+    </xacro:if>
     <!-- GRIPPER RIGHT -->
     <joint name="${prefix}_base_joint_gripper_right" type="prismatic">
@@ -261,32 +277,82 @@
         <limit effort="100" velocity="100"/>
     </joint>
-    <link name="${prefix}_finger_right">
-        <inertial>
-            <mass value="0.052" />
-            <origin xyz="0 0 0.075" />
-            <inertia ixx="2.50e-5" ixy="0.0" ixz="0.0"
-            iyy="2.50e-5" iyz="0.0"
-            izz="2.60e-6"/>
-        </inertial>
-        <visual>
-            <origin xyz="0.0 0 0" rpy="0 0 0" />
-            <geometry>
-                <mesh filename="file://$(find wsg_50_simulation)/meshes/WSG-FMF.stl" scale="0.001 0.001 0.001"/>
-            </geometry>
-            <material name="black">
-            <color rgba="0 0 0 1"/>
-            </material>
-        </visual>
-        <collision>
-            <origin xyz="0 0 0" rpy="0 0 0" />
-            <geometry>
-                <mesh filename="file://$(find wsg_50_simulation)/meshes/WSG-FMF.stl" scale="0.001 0.001 0.001"/>
-            </geometry>
-        </collision>
-        <contact_coefficients kd="1.0" kp="1000.0" mu="0"/>
-    </link>
-    <gazebo reference="${prefix}_finger_right">
-        <material>Gazebo/White</material>
-    </gazebo>
+    <xacro:unless value="${finger_type == 'soft'}">
+        <link name="${prefix}_finger_right">
+            <inertial>
+                <mass value="0.052" />
+                <origin xyz="0 0 0.085" />
+                <inertia ixx="2.50e-5" ixy="0.0" ixz="0.0"
+                iyy="2.50e-5" iyz="0.0"
+                izz="2.60e-6"/>
+            </inertial>
+            <visual>
+                <origin xyz="0.0 0 0" rpy="0 0 0" />
+                <geometry>
+                    <mesh filename="file://$(find wsg_50_simulation)/meshes/WSG-FMF.stl" scale="0.001 0.001 0.001"/>
+                </geometry>
+                <material name="black">
+                <color rgba="0 0 0 1"/>
+                </material>
+            </visual>
+            <collision>
+                <origin xyz="0 0 0" rpy="0 0 0" />
+                <geometry>
+                    <mesh filename="file://$(find wsg_50_simulation)/meshes/WSG-FMF.stl" scale="0.001 0.001 0.001"/>
+                </geometry>
+            </collision>
+            <contact_coefficients kd="1.0" kp="1000.0" mu="0"/>
+        </link>
+        <gazebo reference="${prefix}_finger_right">
+            <material>Gazebo/Black</material>
+        </gazebo>
+    </xacro:unless>
+    <xacro:if value="${finger_type == 'soft'}">
+        <link name="${prefix}_finger_right">
+            <inertial>
+                <mass value="0.052" />
+                <origin xyz="0 0 0" />
+                <inertia ixx="2.50e-5" ixy="0.0" ixz="0.0"
+                        iyy="2.50e-5" iyz="0.0"
+                        izz="2.60e-6"/>
+            </inertial>
+            <!-- Visual for finger_base -->
+            <visual>
+                <origin xyz="0 0 -0.023" rpy="-1.5708 0 0" />
+                <geometry>
+                    <mesh filename="file://$(find wsg_50_simulation)/meshes/finger_base.stl" scale="1. 1. 1."/>
+                </geometry>
+                <material name="orange">
+                    <color rgba="0.98 0.29 0.08 1"/>
+                </material>
+            </visual>
+            <!-- Visual for finger_body -->
+            <visual>
+                <origin xyz="0 0.013 0.078" rpy="3.14 0 3.14" />
+                <geometry>
+                    <mesh filename="file://$(find wsg_50_simulation)/meshes/finger_body.stl" scale="1. 1. 1."/>
+                </geometry>
+                <material name="orange">
+                    <color rgba="0.98 0.29 0.08 1"/>
+                </material>
+            </visual>
+            <!-- Collision -->
+            <collision>
+                <origin xyz="0 0 -0.023" rpy="-1.5708 0 0" />
+                <geometry>
+                    <mesh filename="file://$(find wsg_50_simulation)/meshes/finger_base.stl" scale="1. 1. 1."/>
+                </geometry>
+            </collision>
+            <collision>
+                <origin xyz="0 0.013 0.078" rpy="3.14 0 3.14" />
+                <geometry>
+                    <mesh filename="file://$(find wsg_50_simulation)/meshes/finger_body.stl" scale="1. 1. 1."/>
+                </geometry>
+            </collision>
+            <contact_coefficients kd="1.0" kp="1000.0" mu="0"/>
+        </link>
+        <gazebo reference="${prefix}_finger_right">
+            <material>Gazebo/Orange</material>
+        </gazebo>
+    </xacro:if>
     <ros2_control name="${prefix}" type="system">
         <xacro:unless value="${real_hardware}">

Commit message: adding pal finger

File: wsg_50_simulation/urdf/wsg50.urdf.xacro (robot description, xacro)
@@ -6,5 +6,5 @@
     <xacro:include filename="$(find wsg_50_simulation)/urdf/wsg_50.urdf.xacro" />
     <link name="base_link"/>
-    <xacro:wsg_50_xacro prefix="wsg50" parent="base_link" finger_length="0.023" finger_tip="0.0" sim_standalone="$(arg sim_standalone)" real_hardware="$(arg real_hardware)" finger_type="soft">
+    <xacro:wsg_50_xacro prefix="wsg50" parent="base_link" finger_length="0.023" finger_tip="0.0" sim_standalone="$(arg sim_standalone)" real_hardware="$(arg real_hardware)" finger_type="pal">
         <origin xyz="0 0 0.1" rpy="0 0 0"/>
     </xacro:wsg_50_xacro>

File: wsg_50_simulation/urdf/wsg_50.urdf.xacro (robot description, xacro)
@@ -4,5 +4,5 @@
 <!-- finger_tip:    Offset of finger tip along fingers' motion direction.
                     Use e.g. for single contact point tip on finger. (default 0) -->
-<xacro:macro name="wsg_50_xacro" params="prefix parent finger_length finger_tip *origin sim_standalone:=false real_hardware:=false finger_type:='soft' config_file:=${xacro.load_yaml('$(find wsg_50_driver)/config/wsg50_setup.yaml')}">
+<xacro:macro name="wsg_50_xacro" params="prefix parent finger_length finger_tip *origin sim_standalone:=false real_hardware:=false finger_type:='pal' config_file:=${xacro.load_yaml('$(find wsg_50_driver)/config/wsg50_setup.yaml')}">
     <link name="${prefix}_base"/>
     <joint name="${prefix}_base_joint" type="fixed">
@@ -149,7 +149,8 @@
         <dynamics friction="100" damping="100" />
         <axis xyz="1 0 0"/>
+        <origin xyz="0 0 0" rpy="0 0 0" />
         <limit effort="100" velocity="100"/>
     </joint>
-    <xacro:unless value="${finger_type == 'soft'}">
+    <xacro:if value="${finger_type == 'classic'}">
         <link name="${prefix}_finger_left">
             <inertial>
@@ -180,5 +181,5 @@
             <material>Gazebo/Black</material>
         </gazebo>
-    </xacro:unless>
+    </xacro:if>
     <xacro:if value="${finger_type == 'soft'}">
         <link name="${prefix}_finger_left">
@@ -227,4 +228,52 @@
         <gazebo reference="${prefix}_finger_left">
             <material>Gazebo/Orange</material>
+        </gazebo>
+    </xacro:if>
+    <xacro:if value="${finger_type == 'pal'}">
+        <link name="${prefix}_finger_left">
+            <inertial>
+                <mass value="0.052" />
+                <origin xyz="0 0 0" />
+                <inertia ixx="2.50e-5" ixy="0.0" ixz="0.0"
+                        iyy="2.50e-5" iyz="0.0"
+                        izz="2.60e-6"/>
+            </inertial>
+            <!-- Visual for finger_base -->
+            <visual>
+                <origin xyz="0 0.015 0.1025" rpy="-1.5708 0 -3.14" />
+                <geometry>
+                    <mesh filename="file://$(find wsg_50_simulation)/meshes/mounting-pal.stl" scale="0.001 0.001 0.001"/>
+                </geometry>
+                <material name="black">
+                    <color rgba="0 0 0 1"/>
+                </material>
+            </visual>
+            <!-- Visual for finger_body -->
+            <visual>
+                <origin xyz="0 -0.002 0.0955" rpy="1.5708 0 -1.5708" />
+                <geometry>
+                    <mesh filename="file://$(find wsg_50_simulation)/meshes/finger-PAL.stl" scale="0.001 0.001 0.001"/>
+                </geometry>
+                <material name="black">
+                    <color rgba="0 0 0 1"/>
+                </material>
+            </visual>
+            <!-- Collision -->
+            <collision>
+                <origin xyz="0 0.015 0.1025" rpy="-1.5708 0 -3.14" />
+                <geometry>
+                    <mesh filename="file://$(find wsg_50_simulation)/meshes/mounting-pal.stl" scale="0.001 0.001 0.001"/>
+                </geometry>
+            </collision>
+            <collision>
+                <origin xyz="0 -0.002 0.0955" rpy="1.5708 0 -1.5708" />
+                <geometry>
+                    <mesh filename="file://$(find wsg_50_simulation)/meshes/finger-PAL.stl" scale="0.001 0.001 0.001"/>
+                </geometry>
+            </collision>
+            <contact_coefficients kd="1.0" kp="1000.0" mu="0"/>
+        </link>
+        <gazebo reference="${prefix}_finger_left">
+            <material>Gazebo/Black</material>
         </gazebo>
     </xacro:if>
@@ -277,5 +326,5 @@
         <limit effort="100" velocity="100"/>
     </joint>
-    <xacro:unless value="${finger_type == 'soft'}">
+    <xacro:if value="${finger_type == 'classic'}">
         <link name="${prefix}_finger_right">
             <inertial>
@@ -306,5 +355,5 @@
             <material>Gazebo/Black</material>
         </gazebo>
-    </xacro:unless>
+    </xacro:if>
     <xacro:if value="${finger_type == 'soft'}">
         <link name="${prefix}_finger_right">
@@ -353,4 +402,52 @@
         <gazebo reference="${prefix}_finger_right">
             <material>Gazebo/Orange</material>
+        </gazebo>
+    </xacro:if>
+    <xacro:if value="${finger_type == 'pal'}">
+        <link name="${prefix}_finger_right">
+            <inertial>
+                <mass value="0.052" />
+                <origin xyz="0 0 0" />
+                <inertia ixx="2.50e-5" ixy="0.0" ixz="0.0"
+                        iyy="2.50e-5" iyz="0.0"
+                        izz="2.60e-6"/>
+            </inertial>
+            <!-- Visual for finger_base -->
+            <visual>
+                <origin xyz="0 0.015 0.1025" rpy="-1.5708 0 3.14" />
+                <geometry>
+                    <mesh filename="file://$(find wsg_50_simulation)/meshes/mounting-pal.stl" scale="0.001 0.001 0.001"/>
+                </geometry>
+                <material name="black">
+                    <color rgba="0 0 0 1"/>
+                </material>
+            </visual>
+            <!-- Visual for finger_body -->
+            <visual>
+                <origin xyz="0 -0.002 0.0955" rpy="1.5708 0 -1.5708" />
+                <geometry>
+                    <mesh filename="file://$(find wsg_50_simulation)/meshes/finger-PAL.stl" scale="0.001 0.001 0.001"/>
+                </geometry>
+                <material name="black">
+                    <color rgba="0 0 0 1"/>
+                </material>
+            </visual>
+            <!-- Collision -->
+            <collision>
+                <origin xyz="0 0.015 0.1025" rpy="-1.5708 0 -3.14" />
+                <geometry>
+                    <mesh filename="file://$(find wsg_50_simulation)/meshes/mounting-pal.stl" scale="0.001 0.001 0.001"/>
+                </geometry>
+            </collision>
+            <collision>
+                <origin xyz="0 -0.002 0.0955" rpy="1.5708 0 -1.5708" />
+                <geometry>
+                    <mesh filename="file://$(find wsg_50_simulation)/meshes/finger-PAL.stl" scale="0.001 0.001 0.001"/>
+                </geometry>
+            </collision>
+            <contact_coefficients kd="1.0" kp="1000.0" mu="0"/>
+        </link>
+        <gazebo reference="${prefix}_finger_left">
+            <material>Gazebo/Black</material>
         </gazebo>
     </xacro:if>
